Commit message: fix rviz2 display

File: ROS2/R5_ws/src/ARX_R5_ros2_V7/arx_r5_controller/urdf/R5_master.urdf (robot description, URDF)
Before this commit: robot r5_urdf, 7 links, 6 joints
Links:
- link base_link: geometry collision mesh filename=package://r5_urdf/meshes/base_link.STL; visual mesh filename=package://r5_urdf/meshes/base_link.STL
